Commit message: system rebuild

File: ros2_ws/build/owl_description/urdf/robot.xacro (robot description, xacro)
@@ -1 +1 @@
-/home/aaditya/OWL_Sorting/ros2_ws/src/owl_description/urdf/robot.xacro
+/home/vardan/OWL_Sorting/ros2_ws/src/owl_description/urdf/robot.xacro

File: ros2_ws/build/owl_gazebo/urdf/gazebo_plugins.xacro (robot description, xacro)
@@ -1 +1 @@
-/home/aaditya/OWL_Sorting/ros2_ws/src/owl_gazebo/urdf/gazebo_plugins.xacro
+/home/vardan/OWL_Sorting/ros2_ws/src/owl_gazebo/urdf/gazebo_plugins.xacro

File: ros2_ws/build/owl_gazebo/urdf/sim_gazebo.xacro (robot description, xacro)
@@ -1 +1 @@
-/home/aaditya/OWL_Sorting/ros2_ws/src/owl_gazebo/urdf/sim_gazebo.xacro
+/home/vardan/OWL_Sorting/ros2_ws/src/owl_gazebo/urdf/sim_gazebo.xacro

File: ros2_ws/install/owl_description/share/owl_description/urdf/robot.xacro (robot description, xacro)
@@ -1 +1 @@
-/home/aaditya/OWL_Sorting/ros2_ws/build/owl_description/urdf/robot.xacro
+/home/vardan/OWL_Sorting/ros2_ws/build/owl_description/urdf/robot.xacro

File: ros2_ws/install/owl_gazebo/share/owl_gazebo/urdf/gazebo_plugins.xacro (robot description, xacro)
@@ -1 +1 @@
-/home/aaditya/OWL_Sorting/ros2_ws/build/owl_gazebo/urdf/gazebo_plugins.xacro
+/home/vardan/OWL_Sorting/ros2_ws/build/owl_gazebo/urdf/gazebo_plugins.xacro

File: ros2_ws/install/owl_gazebo/share/owl_gazebo/urdf/sim_gazebo.xacro (robot description, xacro)
@@ -1 +1 @@
-/home/aaditya/OWL_Sorting/ros2_ws/build/owl_gazebo/urdf/sim_gazebo.xacro
+/home/vardan/OWL_Sorting/ros2_ws/build/owl_gazebo/urdf/sim_gazebo.xacro

File: ros2_ws/src/owl_gazebo/urdf/gazebo_plugins.xacro (robot description, xacro)
@@ -41,21 +41,3 @@
 	  <xacro:simple_transmission joint_name="W3J" actuator_name="W3J_motor"/>
 	</xacro:macro>
-	<gazebo reference="base_link">
-	    <material>Gazebo/Silver</material>
-    </gazebo>
-	<gazebo reference="shoulder_link">
-	    <material>Gazebo/Silver</material>
-    </gazebo>
-	<gazebo reference="link1">
-	    <material>Gazebo/Gray</material>
-    </gazebo>
-	<gazebo reference="elbow_link">
-	    <material>Gazebo/Silver</material>
-    </gazebo>
-	<gazebo reference="link2">
-	    <material>Gazebo/Gray</material>
-    </gazebo>
-	<gazebo reference="w2w3_link">
-	    <material>Gazebo/Gray</material>
-    </gazebo>
 </robot>
