Commit message: urdf's up and running

File: ros2_ws/src/owl_description/urdf/robot.xacro (robot description, xacro)
@@ -31,5 +31,5 @@
       <geometry>
         <mesh
-          filename="package://owl_description/meshes/base_link.STL" />
+          filename="$(find owl_description)/meshes/base_link.STL" />
       </geometry>
       <material
@@ -45,5 +45,5 @@
       <geometry>
         <mesh
-          filename="package://owl_description/meshes/base_link.STL" />
+          filename="$(find owl_description)/meshes/base_link.STL" />
       </geometry>
     </collision>
@@ -71,19 +71,19 @@
       <geometry>
         <mesh
-          filename="package://owl_description/meshes/shoulder_link.STL" />
-      </geometry>
-      <material
-        name="">
-        <color
-          rgba="0.79216 0.81961 0.93333 1" />
-      </material>
-    </visual>
-    <collision>
-      <origin
-        xyz="0 0 0"
-        rpy="0 0 0" />
-      <geometry>
-        <mesh
-          filename="package://owl_description/meshes/shoulder_link.STL" />
+          filename="$(find owl_description)/meshes/shoulder_link.STL" />
+      </geometry>
+      <material
+        name="">
+        <color
+          rgba="0.79216 0.81961 0.93333 1" />
+      </material>
+    </visual>
+    <collision>
+      <origin
+        xyz="0 0 0"
+        rpy="0 0 0" />
+      <geometry>
+        <mesh
+          filename="$(find owl_description)/meshes/shoulder_link.STL" />
       </geometry>
     </collision>
@@ -125,19 +125,19 @@
       <geometry>
         <mesh
-          filename="package://owl_description/meshes/link1.STL" />
-      </geometry>
-      <material
-        name="">
-        <color
-          rgba="0.79216 0.81961 0.93333 1" />
-      </material>
-    </visual>
-    <collision>
-      <origin
-        xyz="0 0 0"
-        rpy="0 0 0" />
-      <geometry>
-        <mesh
-          filename="package://owl_description/meshes/link1.STL" />
+          filename="$(find owl_description)/meshes/link1.STL" />
+      </geometry>
+      <material
+        name="">
+        <color
+          rgba="0.79216 0.81961 0.93333 1" />
+      </material>
+    </visual>
+    <collision>
+      <origin
+        xyz="0 0 0"
+        rpy="0 0 0" />
+      <geometry>
+        <mesh
+          filename="$(find owl_description)/meshes/link1.STL" />
       </geometry>
     </collision>
@@ -179,19 +179,19 @@
       <geometry>
         <mesh
-          filename="package://owl_description/meshes/elbow_link.STL" />
-      </geometry>
-      <material
-        name="">
-        <color
-          rgba="0.79216 0.81961 0.93333 1" />
-      </material>
-    </visual>
-    <collision>
-      <origin
-        xyz="0 0 0"
-        rpy="0 0 0" />
-      <geometry>
-        <mesh
-          filename="package://owl_description/meshes/elbow_link.STL" />
+          filename="$(find owl_description)/meshes/elbow_link.STL" />
+      </geometry>
+      <material
+        name="">
+        <color
+          rgba="0.79216 0.81961 0.93333 1" />
+      </material>
+    </visual>
+    <collision>
+      <origin
+        xyz="0 0 0"
+        rpy="0 0 0" />
+      <geometry>
+        <mesh
+          filename="$(find owl_description)/meshes/elbow_link.STL" />
       </geometry>
     </collision>
@@ -233,19 +233,19 @@
       <geometry>
         <mesh
-          filename="package://owl_description/meshes/link2.STL" />
-      </geometry>
-      <material
-        name="">
-        <color
-          rgba="0.79216 0.81961 0.93333 1" />
-      </material>
-    </visual>
-    <collision>
-      <origin
-        xyz="0 0 0"
-        rpy="0 0 0" />
-      <geometry>
-        <mesh
-          filename="package://owl_description/meshes/link2.STL" />
+          filename="$(find owl_description)/meshes/link2.STL" />
+      </geometry>
+      <material
+        name="">
+        <color
+          rgba="0.79216 0.81961 0.93333 1" />
+      </material>
+    </visual>
+    <collision>
+      <origin
+        xyz="0 0 0"
+        rpy="0 0 0" />
+      <geometry>
+        <mesh
+          filename="$(find owl_description)/meshes/link2.STL" />
       </geometry>
     </collision>
@@ -287,19 +287,19 @@
       <geometry>
         <mesh
-          filename="package://owl_description/meshes/w2w3_link.STL" />
-      </geometry>
-      <material
-        name="">
-        <color
-          rgba="0.79216 0.81961 0.93333 1" />
-      </material>
-    </visual>
-    <collision>
-      <origin
-        xyz="0 0 0"
-        rpy="0 0 0" />
-      <geometry>
-        <mesh
-          filename="package://owl_description/meshes/w2w3_link.STL" />
+          filename="$(find owl_description)/meshes/w2w3_link.STL" />
+      </geometry>
+      <material
+        name="">
+        <color
+          rgba="0.79216 0.81961 0.93333 1" />
+      </material>
+    </visual>
+    <collision>
+      <origin
+        xyz="0 0 0"
+        rpy="0 0 0" />
+      <geometry>
+        <mesh
+          filename="$(find owl_description)/meshes/w2w3_link.STL" />
       </geometry>
     </collision>
@@ -341,19 +341,19 @@
       <geometry>
         <mesh
-          filename="package://owl_description/meshes/end_effector_link.STL" />
-      </geometry>
-      <material
-        name="">
-        <color
-          rgba="0.79216 0.81961 0.93333 1" />
-      </material>
-    </visual>
-    <collision>
-      <origin
-        xyz="0 0 0"
-        rpy="0 0 0" />
-      <geometry>
-        <mesh
-          filename="package://owl_description/meshes/end_effector_link.STL" />
+          filename="$(find owl_description)/meshes/end_effector_link.STL" />
+      </geometry>
+      <material
+        name="">
+        <color
+          rgba="0.79216 0.81961 0.93333 1" />
+      </material>
+    </visual>
+    <collision>
+      <origin
+        xyz="0 0 0"
+        rpy="0 0 0" />
+      <geometry>
+        <mesh
+          filename="$(find owl_description)/meshes/end_effector_link.STL" />
       </geometry>
     </collision>

Commit message: this is final branch

File: ros2_ws/src/owl_description/urdf/robot.xacro (robot description, xacro)
@@ -5,5 +5,5 @@
     name="virtual_joint"
     type="fixed">
-    <origin xyz="0 0 0.0" rpy="0 0 0" />
+    <origin xyz="0 0 0" rpy="0 0 0" />
     <parent link="world" />
     <child link="base_link" />

Commit message: major updates in urdf and other files

File: ros2_ws/src/owl_description/urdf/robot.xacro (robot description, xacro)
@@ -1,421 +1,9 @@
-<?xml version="1.0" encoding="utf-8"?>
-<robot xmlns:xacro="http://www.ros.org/wiki/xacro" name="owl_description">
-  <link name="world" />
-  <joint
-    name="virtual_joint"
-    type="fixed">
-    <origin xyz="0 0 0" rpy="0 0 0" />
-    <parent link="world" />
-    <child link="base_link" />
-  </joint>
-  <link
-    name="base_link">
-    <inertial>
-      <origin
-        xyz="2.7395E-05 -0.01813 4.3722E-05"
-        rpy="0 0 0" />
-      <mass
-        value="2.39" />
-      <inertia
-        ixx="0.0060063"
-        ixy="-2.5541E-15"
-        ixz="-2.5603E-07"
-        iyy="0.0095451"
-        iyz="5.1619E-15"
-        izz="0.006006" />
-    </inertial>
-    <visual>
-      <origin
-        xyz="0 0 0"
-        rpy="0 0 0" />
-      <geometry>
-        <mesh
-          filename="$(find owl_description)/meshes/base_link.STL" />
-      </geometry>
-      <material
-        name="">
-        <color
-          rgba="0.89804 0.91765 0.92941 1" />
-      </material>
-    </visual>
-    <collision>
-      <origin
-        xyz="0 0 0"
-        rpy="0 0 0" />
-      <geometry>
-        <mesh
-          filename="$(find owl_description)/meshes/base_link.STL" />
-      </geometry>
-    </collision>
-  </link>
-  <link
-    name="shoulder_link">
-    <inertial>
-      <origin
-        xyz="0.00042134 0.034391 -0.10382"
-        rpy="0 0 0" />
-      <mass
-        value="4.613" />
-      <inertia
-        ixx="0.0035279"
-        ixy="-5.6452E-06"
-        ixz="-9.4882E-07"
-        iyy="0.0046955"
-        iyz="0.00045199"
-        izz="0.0048177" />
-    </inertial>
-    <visual>
-      <origin
-        xyz="0 0 0"
-        rpy="0 0 0" />
-      <geometry>
-        <mesh
-          filename="$(find owl_description)/meshes/shoulder_link.STL" />
-      </geometry>
-      <material
-        name="">
-        <color
-          rgba="0.79216 0.81961 0.93333 1" />
-      </material>
-    </visual>
-    <collision>
-      <origin
-        xyz="0 0 0"
-        rpy="0 0 0" />
-      <geometry>
-        <mesh
-          filename="$(find owl_description)/meshes/shoulder_link.STL" />
-      </geometry>
-    </collision>
-  </link>
-  <joint
-    name="BJ"
-    type="continuous">
-    <origin
-      xyz="0 0 0"
-      rpy="-3.1416 0 -1.574" />
-    <parent
-      link="base_link" />
-    <child
-      link="shoulder_link" />
-    <axis
-      xyz="0 0 1" />
-    <limit effort="500" velocity="0.873" lower="-2.0944" upper="2.0944"/>
-  </joint>
-  <link
-    name="link1">
-    <inertial>
-      <origin
-        xyz=" 0.17795 0.00011012 -0.085428"
-        rpy="0 0 0" />
-      <mass
-        value="9.431" />
-      <inertia
-        ixx="0.0052455"
-        ixy="1.4977E-05"
-        ixz="2.6778E-05"
-        iyy="0.028778"
-        iyz="-3.8624E-06"
-        izz="0.032177" />
-    </inertial>
-    <visual>
-      <origin
-        xyz="0 0 0"
-        rpy="0 0 0" />
-      <geometry>
-        <mesh
-          filename="$(find owl_description)/meshes/link1.STL" />
-      </geometry>
-      <material
-        name="">
-        <color
-          rgba="0.79216 0.81961 0.93333 1" />
-      </material>
-    </visual>
-    <collision>
-      <origin
-        xyz="0 0 0"
-        rpy="0 0 0" />
-      <geometry>
-        <mesh
-          filename="$(find owl_description)/meshes/link1.STL" />
-      </geometry>
-    </collision>
-  </link>
-  <joint
-    name="SJ"
-    type="continuous">
-    <origin
-      xyz="0.00018339 0.066603 -0.1405"
-      rpy="0.58944 1.5675 -0.983" />
-    <parent
-      link="shoulder_link" />
-    <child
-      link="link1" />
-    <axis
-      xyz="0.0027142 -0.0011243 1" />
-    <limit effort="500" velocity="0.873" lower="-1.6" upper="1.6"/>
-  </joint>
-  <link
-    name="elbow_link">
-    <inertial>
-      <origin
-        xyz="0.00023616 -0.028792 -0.029823"
-        rpy="0 0 0" />
-      <mass
-        value="4.613" />
-      <inertia
-        ixx="0.0023499"
-        ixy="-2.7675E-06"
-        ixz="-4.1087E-07"
-        iyy="0.0030181"
-        iyz="-0.00026183"
-        izz="0.0035661" />
-    </inertial>
-    <visual>
-      <origin
-        xyz="0 0 0"
-        rpy="0 0 0" />
-      <geometry>
-        <mesh
-          filename="$(find owl_description)/meshes/elbow_link.STL" />
-      </geometry>
-      <material
-        name="">
-        <color
-          rgba="0.79216 0.81961 0.93333 1" />
-      </material>
-    </visual>
-    <collision>
-      <origin
-        xyz="0 0 0"
-        rpy="0 0 0" />
-      <geometry>
-        <mesh
-          filename="$(find owl_description)/meshes/elbow_link.STL" />
-      </geometry>
-    </collision>
-  </link>
-  <joint
-    name="EJ"
-    type="continuous">
-    <origin
-      xyz="0.35575 0 -0.00096557"
-      rpy="3.1389 -0.0018334 -1.5781" />
-    <parent
-      link="link1" />
-    <child
-      link="elbow_link" />
-    <axis
-      xyz="0 0 1" />
-    <limit effort="500" velocity="0.873" lower="-1.57" upper="3.14"/>
-  </joint>
-  <link
-    name="link2">
-    <inertial>
-      <origin
-        xyz="0.00015054 -0.075078 0.13834"
-        rpy="0 0 0" />
-      <mass
-        value="2.4407" />
-      <inertia
-        ixx="0.009134"
-        ixy="-3.9978E-06"
-        ixz="-4.8015E-06"
-        iyy="0.010823"
-        iyz="0.00068065"
-        izz="0.0041094" />
-    </inertial>
-    <visual>
-      <origin
-        xyz="0 0 0"
-        rpy="0 0 0" />
-      <geometry>
-        <mesh
-          filename="$(find owl_description)/meshes/link2.STL" />
-      </geometry>
-      <material
-        name="">
-        <color
-          rgba="0.79216 0.81961 0.93333 1" />
-      </material>
-    </visual>
-    <collision>
-      <origin
-        xyz="0 0 0"
-        rpy="0 0 0" />
-      <geometry>
-        <mesh
-          filename="$(find owl_description)/meshes/link2.STL" />
-      </geometry>
-    </collision>
-  </link>
-  <joint
-    name="W1J"
-    type="continuous">
-    <origin
-      xyz="0.00019567 -0.079361 -0.066603"
-      rpy="1.5708 -0.0023608 0" />
-    <parent
-      link="elbow_link" />
-    <child
-      link="link2" />
-    <axis
-      xyz="0 0 -1" />
-    <limit effort="500" velocity="0.873" lower="-2.84489" upper="2.84489"/>
-  </joint>
-  <link
-    name="w2w3_link">
-    <inertial>
-      <origin
-        xyz="0.00025923 0.029764 0.027271"
-        rpy="0 0 0" />
-      <mass
-        value="3.118" />
-      <inertia
-        ixx="0.0014884"
-        ixy="2.1526E-06"
-        ixz="6.6731E-06"
-        iyy="0.0016882"
-        iyz="0.0001816"
-        izz="0.0019291" />
-    </inertial>
-    <visual>
-      <origin
-        xyz="0 0 0"
-        rpy="0 0 0" />
-      <geometry>
-        <mesh
-          filename="$(find owl_description)/meshes/w2w3_link.STL" />
-      </geometry>
-      <material
-        name="">
-        <color
-          rgba="0.79216 0.81961 0.93333 1" />
-      </material>
-    </visual>
-    <collision>
-      <origin
-        xyz="0 0 0"
-        rpy="0 0 0" />
-      <geometry>
-        <mesh
-          filename="$(find owl_description)/meshes/w2w3_link.STL" />
-      </geometry>
-    </collision>
-  </link>
-  <joint
-    name="W2J"
-    type="continuous">
-    <origin
-      xyz="0 0 0.27639"
-      rpy="2.745 -1.5667 -1.1726" />
-    <parent
-      link="link2" />
-    <child
-      link="w2w3_link" />
-    <axis
-      xyz="0.0037507 -0.00083382 0.99999" />
-    <limit effort="500" velocity="0.873" lower="-1.6" upper="2.1"/>
-  </joint>
-  <link
-    name="end_effector_link">
-    <inertial>
-      <origin
-        xyz="2.2451E-05 -0.00060487 0.098537"
-        rpy="0 0 0" />
-      <mass
-        value="0.188" />
-      <inertia
-        ixx="0.00017935"
-        ixy="-3.2299E-08"
-        ixz="-2.1374E-07"
-        iyy="0.00017907"
-        iyz="-4.545E-07"
-        izz="0.00025742" />
-    </inertial>
-    <visual>
-      <origin
-        xyz="0 0 0"
-        rpy="0 0 0" />
-      <geometry>
-        <mesh
-          filename="$(find owl_description)/meshes/end_effector_link.STL" />
-      </geometry>
-      <material
-        name="">
-        <color
-          rgba="0.79216 0.81961 0.93333 1" />
-      </material>
-    </visual>
-    <collision>
-      <origin
-        xyz="0 0 0"
-        rpy="0 0 0" />
-      <geometry>
-        <mesh
-          filename="$(find owl_description)/meshes/end_effector_link.STL" />
-      </geometry>
-    </collision>
-  </link>
-  <joint
-    name="W3J"
-    type="continuous">
-    <origin
-      xyz="0 0 0"
-      rpy="-1.2578 -1.5668 -0.31786" />
-    <limit effort="500" velocity="0.873" lower="-3.1" upper="3.1"/>
-    <parent
-      link="w2w3_link" />
-    <child
-      link="end_effector_link" />
-    <axis
-      xyz="0 0 1" />
-  </joint>
-  <xacro:arg name="tcp_xyz" default="0 0 0" />
-  <xacro:arg name="tcp_rpy" default="0 0 0" />
-  <xacro:arg name="payload_mass" default="0" />
-  <xacro:arg name="payload_cog" default="0 0 0" />
-  <xacro:arg name="payload_radius" default="0" />
-  <xacro:arg name="payload_ixx" default="0" />
-  <xacro:arg name="payload_ixy" default="0" />
-  <xacro:arg name="payload_ixz" default="0" />
-  <xacro:arg name="payload_iyy" default="0" />
-  <xacro:arg name="payload_iyz" default="0" />
-  <xacro:arg name="payload_izz" default="0" />
-  <link name="tool_mount">
-    <inertial>
-      <origin xyz="$(arg payload_cog)" rpy="0 0 0" />
-      <mass value="$(arg payload_mass)" />
-      <inertia ixx="$(arg payload_ixx)" ixy="$(arg payload_ixy)" ixz="$(arg payload_ixz)" iyy="$(arg payload_iyy)" iyz="$(arg payload_iyz)" izz="$(arg payload_izz)" />
-    </inertial>
-    <visual>
-      <origin xyz="$(arg payload_cog)" rpy="0 0 0" />
-      <geometry>
-        <sphere radius="$(arg payload_radius)"/>
-      </geometry>
-      <material name="green">
-          <color rgba="0 1 0 1"/>
-      </material>
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
File: ros2_ws/src/owl_gazebo/urdf/gazebo_plugins.xacro (robot description, xacro)
@@ -20,7 +20,27 @@
 <!-- This macro call for adding gazebo control to the urdf -->
 	<xacro:macro name="gazebo_control">
-	  <gazebo>
-	    <plugin name="gazebo_ros_control" filename="libgazebo_ros_control.so">
-	    </plugin>
+	  <gazebo reference="camera_link">
+	  	<sensor name="camera" type="camera">
+		<camera>
+		<horizontal_fov>1.0472</horizontal_fov>
+		<image>
+			<width>640</width>
+			<height>480</height>
+			<format>R8G8B8</format>
+		</image>
+		<clip>
+			<near>0.1</near>
+			<far>100</far>
+		</clip>
+		</camera>
+			<plugin name="gazebo_ros_camera" filename="libgazebo_ros_camera.so">
+			<robotNamespace>/owr_6.5</robotNamespace>
+			<cameraName>camera</cameraName>
+			<imageTopicName>/camera/image_raw</imageTopicName>
+			<cameraInfoTopicName>/camera/camera_info</cameraInfoTopicName>
+			<updateRate>30.0</updateRate>
+			<frameName>camera_link</frameName>
+		</plugin>
+	</sensor>
 	  </gazebo>
 	  <!-- Applying gazebo_self_collide macro -->
@@ -41,3 +61,4 @@
 	  <xacro:simple_transmission joint_name="W3J" actuator_name="W3J_motor"/>
 	</xacro:macro>
+    <!--Add camera sensor to end_effector_link -->
 </robot>

File: ros2_ws/src/owl_gazebo/urdf/sim_gazebo.xacro (robot description, xacro)
@@ -1,9 +1,9 @@
 <?xml version="1.0"?>
 <robot name="owl_description" xmlns:xacro="http://wiki.ros.org/xacro">
-    <xacro:include filename="$(find owl_description)/urdf/robot.xacro"/>
+    <xacro:include filename="$(find owl_description)/urdf/owl.xacro"/>
     <xacro:include filename="$(find owl_gazebo)/urdf/gazebo_plugins.xacro"/>
-    <xacro parent="world">
-        <origin xyz="0.0 0.0 0.55" rpy="0 0 0" />
-    </xacro>
+        <xacro:owl_arm parent="world">
+            <origin xyz="0.0 0.0 0.0" rpy="0 0 0" />
+        </xacro:owl_arm>
     <xacro:gazebo_control/>
 </robot>
