Commit message: camera plugin functional finally

File: ros2_ws/src/owl_gazebo/urdf/gazebo_plugins.xacro (robot description, xacro)
@@ -1,64 +1,78 @@
 <?xml version="1.0" encoding="utf-8"?>
 <robot xmlns:xacro="http://ros.org/wiki/xacro">
-	<xacro:macro name="gazebo_self_collide" params="link_name">
-	    <gazebo reference="${link_name}">
-		<selfCollide>true</selfCollide>
-	    </gazebo>
-	</xacro:macro>
-	<xacro:macro name="simple_transmission" params="joint_name actuator_name">
-	    <transmission name="${joint_name}_trans">
-		<type>transmission_interface/SimpleTransmission</type>
-		<joint name="${joint_name}">
-		    <hardwareInterface>hardware_interface/PositionJointInterface</hardwareInterface>
-		</joint>
-		<actuator name="${actuator_name}">
-		    <hardwareInterface>hardware_interface/PositionJointInterface</hardwareInterface>
-		    <mechanicalReduction>1</mechanicalReduction>
-		</actuator>
-	    </transmission>
-	</xacro:macro>
-<!-- This macro call for adding gazebo control to the urdf -->
-	<xacro:macro name="gazebo_control">
-	  <gazebo reference="camera_link">
-	  	<sensor name="camera" type="camera">
-		<camera>
-		<horizontal_fov>1.0472</horizontal_fov>
-		<image>
-			<width>640</width>
-			<height>480</height>
-			<format>R8G8B8</format>
-		</image>
-		<clip>
-			<near>0.1</near>
-			<far>100</far>
-		</clip>
-		</camera>
-			<plugin name="gazebo_ros_camera" filename="libgazebo_ros_camera.so">
-			<robotNamespace>/owr_6.5</robotNamespace>
-			<cameraName>camera</cameraName>
-			<imageTopicName>/camera/image_raw</imageTopicName>
-			<cameraInfoTopicName>/camera/camera_info</cameraInfoTopicName>
-			<updateRate>30.0</updateRate>
-			<frameName>camera_link</frameName>
-		</plugin>
-	</sensor>
-	  </gazebo>
-	  <!-- Applying gazebo_self_collide macro -->
-	  <xacro:gazebo_self_collide link_name="base_link"/>
-	  <xacro:gazebo_self_collide link_name="shoulder_link"/>
-	  <xacro:gazebo_self_collide link_name="link1"/>
-	  <xacro:gazebo_self_collide link_name="elbow_link"/>
-	  <xacro:gazebo_self_collide link_name="link2"/>
-	  <xacro:gazebo_self_collide link_name="w2w3_link"/>
-	  <xacro:gazebo_self_collide link_name="end_effector_link"/>
-	  <xacro:gazebo_self_collide link_name="tcp"/>
-	  <!-- Applying simple_transmission macro -->
-	  <xacro:simple_transmission joint_name="BJ" actuator_name="BJ_motor"/>
-	  <xacro:simple_transmission joint_name="SJ" actuator_name="SJ_motor"/>
-	  <xacro:simple_transmission joint_name="EJ" actuator_name="EJ_motor"/>
-	  <xacro:simple_transmission joint_name="W1J" actuator_name="W1J_motor"/>
-	  <xacro:simple_transmission joint_name="W2J" actuator_name="W2J_motor"/>
-	  <xacro:simple_transmission joint_name="W3J" actuator_name="W3J_motor"/>
-	</xacro:macro>
-    <!--Add camera sensor to end_effector_link -->
+    <xacro:macro name="gazebo_self_collide" params="link_name">
+        <gazebo reference="${link_name}">
+            <selfCollide>true</selfCollide>
+        </gazebo>
+    </xacro:macro>
+    <xacro:macro name="simple_transmission" params="joint_name actuator_name">
+        <transmission name="${joint_name}_trans">
+            <type>transmission_interface/SimpleTransmission</type>
+            <joint name="${joint_name}">
+                <hardwareInterface>hardware_interface/PositionJointInterface</hardwareInterface>
+            </joint>
+            <actuator name="${actuator_name}">
+                <hardwareInterface>hardware_interface/PositionJointInterface</hardwareInterface>
+                <mechanicalReduction>1</mechanicalReduction>
+            </actuator>
+        </transmission>
+    </xacro:macro>
+    <!-- This macro call for adding gazebo control to the urdf -->
+    <xacro:macro name="gazebo_control">
+        <gazebo reference="camera_link">
+            <sensor name="camera" type="camera">
+                <camera>
+                    <horizontal_fov>1.0472</horizontal_fov>
+                    <image>
+                        <width>640</width>
+                        <height>480</height>
+                        <format>R8G8B8</format>
+                    </image>
+                    <clip>
+                        <near>0.1</near>
+                        <far>100</far>
+                    </clip>
+                    <noise>
+                        <type>gaussian</type>
+                        <mean>0.0</mean>
+                        <stddev>0.007</stddev>
+                    </noise>
+                </camera>
+                <always_on>1</always_on>
+                <update_rate>30</update_rate>
+				<!--  -->
+                <visualize>true</visualize>
+                <plugin name="camera_controller" filename="libgazebo_ros_camera.so">
+                    <alwaysOn>true</alwaysOn>
+                    <updateRate>0.0</updateRate>
+                    <cameraName>owr_6.5/camera</cameraName>
+                    <imageTopicName>image_raw</imageTopicName>
+                    <cameraInfoTopicName>camera_info</cameraInfoTopicName>
+                    <frameName>camera_link</frameName>
+                    <hackBaseline>0.07</hackBaseline>
+                    <distortionK1>0.0</distortionK1>
+                    <distortionK2>0.0</distortionK2>
+                    <distortionK3>0.0</distortionK3>
+                    <distortionT1>0.0</distortionT1>
+                    <distortionT2>0.0</distortionT2>
+                </plugin>
+            </sensor>
+        </gazebo>
+        <!-- Applying gazebo_self_collide macro -->
+        <xacro:gazebo_self_collide link_name="base_link"/>
+        <xacro:gazebo_self_collide link_name="shoulder_link"/>
+        <xacro:gazebo_self_collide link_name="link1"/>
+        <xacro:gazebo_self_collide link_name="elbow_link"/>
+        <xacro:gazebo_self_collide link_name="link2"/>
+        <xacro:gazebo_self_collide link_name="w2w3_link"/>
+        <xacro:gazebo_self_collide link_name="end_effector_link"/>
+        <xacro:gazebo_self_collide link_name="tcp"/>
+        <!-- Applying simple_transmission macro -->
+        <xacro:simple_transmission joint_name="BJ" actuator_name="BJ_motor"/>
+        <xacro:simple_transmission joint_name="SJ" actuator_name="SJ_motor"/>
+        <xacro:simple_transmission joint_name="EJ" actuator_name="EJ_motor"/>
+        <xacro:simple_transmission joint_name="W1J" actuator_name="W1J_motor"/>
+        <xacro:simple_transmission joint_name="W2J" actuator_name="W2J_motor"/>
+        <xacro:simple_transmission joint_name="W3J" actuator_name="W3J_motor"/>
+    </xacro:macro>
 </robot>
